Commit message: need to refactor; pdff should work on 3D robots

File: urdf/braccio.urdf (robot description, URDF)
Before this commit: robot braccio, 8 links, 7 joints
Links:
- link braccio_base_link: geometry visual mesh filename=package://stl/braccio_base.stl scale=0.001 0.001 0.001
- link elbow_link: geometry visual mesh filename=package://stl/braccio_elbow.stl scale=0.001 0.001 0.001
- link left_gripper_link: geometry visual mesh filename=package://stl/braccio_left_gripper.stl scale=0.001 0.001 0.001
- link right_gripper_link: geometry visual mesh filename=package://stl/braccio_right_gripper.stl scale=0.001 0.001 0.001
- link shoulder_link: geometry visual mesh filename=package://stl/braccio_shoulder.stl scale=0.001 0.001 0.001
- link wrist_pitch_link: geometry visual mesh filename=package://stl/braccio_wrist_pitch.stl scale=0.001 0.001 0.001
- link wrist_roll_link: geometry visual mesh filename=package://stl/braccio_wrist_roll.stl scale=0.001 0.001 0.001
