Commit message: adding braccio urdf loader
Co-authored-by: Prithvi Marwah <prmarwah@users.noreply.github.com>
Co-authored-by: Pranshu Malik <pranshumalik14@gmail.com>

File: src/robot/xacro/braccio_description/urdf/braccio.urdf (robot description, URDF)
Before this commit: robot braccio, 8 links, 7 joints
Links:
- link braccio_base_link: geometry visual mesh filename=package://braccio_description/meshes/braccio_base.stl scale=0.001 0.001 0.001
- link elbow_link: geometry visual mesh filename=package://braccio_description/meshes/braccio_elbow.stl scale=0.001 0.001 0.001
- link left_gripper_link: geometry visual mesh filename=package://braccio_description/meshes/braccio_left_gripper.s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 scale=0.001 0.001 0.001
- link right_gripper_link: geometry visual mesh filename=package://braccio_description/meshes/braccio_right_gripper.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 scale=0.001 0.001 0.001
- link shoulder_link: geometry visual mesh filename=package://braccio_description/meshes/braccio_shoulder.stl scale=0.001 0.001 0.001
- link wrist_pitch_link: geometry visual mesh filename=package://braccio_description/meshes/braccio_wrist_pitch.stl scale=0.001 0.001 0.001
- link wrist_roll_link: geometry visual mesh filename=package://braccio_description/meshes/braccio_wrist_roll.stl scale=0.001 0.001 0.001

Commit message: need to configure urdf with the physical robot joint defaults

File: src/robot/xacro/braccio_description/urdf/braccio.urdf (robot description, URDF)
Before this commit: robot braccio, 8 links, 7 joints
Joints:
- joint gripper_joint: origin xyz=0.010 0 0.03 rpy=0 -0.2967 0 -> xyz=0.010 0 0.03 rpy=0 -1.58 0; type revolute -> fixed
- joint sub_gripper_joint: origin xyz=-0.010 0 0.03 rpy=0 3.4383 0 -> xyz=-0.010 0 0.03 rpy=0 4.62 0; type revolute -> fixed

Commit message: imulation integration done; try pdff in simulation

File: src/robot/xacro/braccio_description/urdf/braccio.urdf (robot description, URDF)
Before this commit: robot braccio, 8 links, 7 joints
Joints:
- joint base_joint: origin xyz=0 0 0 rpy=0 0 0 -> xyz=0 0 0 rpy=0 0 -1.5708

Commit message: changed urdf

File: src/robot/xacro/braccio_description/urdf/braccio.urdf (robot description, URDF)
Before this commit: robot braccio, 8 links, 7 joints
Joints:
- joint wrist_roll_joint: origin xyz=0 0.0 0.06 rpy=0 0 1.5708 -> xyz=0 0.0 0.06 rpy=0 0 0; type revolute -> fixed
